Commit message: Update urdf

File: config/rosbot_xl.urdf (robot description, URDF)
Before this commit: robot rosbot_xl, 12 links, 11 joints
Links:
- removed link velodyne
- removed link velodyne_puck_link
- added link laser
- added link slamtec_rplidar_s1_link, mass 0.105; collision box size=0.0555 0.0555 0.0195; collision cylinder length=0.051 radius=0.02775
Joints:
- removed joint cover_to_velodyne_puck_joint
- removed joint velodyne_puck_to_velodyne_joint
- added joint cover_to_slamtec_rplidar_s1_joint: type fixed, parent cover_link, child slamtec_rplidar_s1_link, origin xyz=0.0 0.0 0.0 rpy=0.0 0.0 0.0
- added joint slamtec_rplidar_s1_to_laser_joint: type fixed, parent slamtec_rplidar_s1_link, child laser, origin xyz=0.0 0.0 0.04 rpy=0.0 0.0 3.141592653589793
